Commit message: X2 demo tooling + sim2real deploy tuning + docs
MuJoCo eval (eval_x2_mujoco.py):
- --motions dance iteration (RSI-reset per clip), --clip name filter
- --record trajectory capture (npz) for sim-vs-real comparison
- manual forward push (P key, head/neck) + difficulty rating keys (E/M/D)
- tolerant checkpoint loader (loads full/stripped .pt without the trl pkg)

Sim2real: x2_ultra.py waist p/r effort 48->36 (PFP-59-60 motor peak) + urdf.

Deploy: new walking_recovery_loose.yaml preset (leg/waist clamps loosened,
waist LPF off); validated on the real robot; documented in tuning README.

Docs: x2_real_robot_test_plan, x2_recovery_robustness_training_plan,
x2_push_test_results, x2_upgraded_demo runbook + dance difficulty ratings
+ demo motion bundle (LFS pointers).

Also snapshots other in-progress tracked changes on this demo branch
(x2_dataset_recorder, x2_kplanner, arm-dynamics config, motion_lib).

Co-Authored-By: Claude Opus 4.8 <noreply@anthropic.com>

File: gear_sonic/data/assets/robot_description/urdf/x2_ultra/x2_ultra.urdf (robot description, URDF)
Before this commit: robot x2t2.5, 41 links, 40 joints
Joints:
- joint left_wrist_pitch_joint: limit lower=-0.558 upper=0.558 effort=4.8 velocity=4.188 -> lower=-0.558 upper=0.558 effort=6.0 velocity=20.944
- joint left_wrist_roll_joint: limit lower=-1.571 upper=0.724 effort=4.8 velocity=4.188 -> lower=-1.571 upper=0.724 effort=6.0 velocity=20.944
- joint right_wrist_pitch_joint: limit lower=-0.558 upper=0.558 effort=4.8 velocity=4.188 -> lower=-0.558 upper=0.558 effort=6.0 velocity=20.944
- joint right_wrist_roll_joint: limit lower=-0.724 upper=1.571 effort=4.8 velocity=4.188 -> lower=-0.724 upper=1.571 effort=6.0 velocity=20.944
